File: hardware/compact/screen-hopper-compact.kicad_pcb (KiCad board)
At the start: 2 copper layers, 82.4 x 58.9 mm, 11 parts, among them J1 USB_A_Host, J2 USB_C_Host, U1 6N137

Commit message: feat: hardware board designs
Parts:
- added U2: USBLC6-2SC6, SOT-23-6, F.Cu at (24.0, 28.0)
- J1: footprint USB_A_Connfly_DS1095 -> USB_A_TE_292303-7_Horizontal
- moved J2 9.99 mm to (6.50, 41.0), turned to -90 degrees
- moved J1 4.73 mm to (10.5, 16.0), turned to -90 degrees
Routing:
- net VBUS1: track 98.7 -> 127.5 mm, vias 2 -> 3
- net USB_DM: track 60.3 -> 74.4 mm, vias 1 -> 2
- net GND1: track 307.1 -> 316.5 mm, vias 0 -> 3
- net USB_DP: track 62.1 -> 70.7 mm, vias 2 -> 1
- net CC2: track 18.6 -> 15.1 mm
- net SER_A2_B3: track 20.5 -> 22.6 mm
- net CC1: track 13.6 -> 14.6 mm
- net SER_A3_B2: track 21.0 -> 20.4 mm
Other:
- board size 82.4 x 58.9 mm -> 88.8 x 58.9 mm

Commit message: [automated commit or incremental update]
Parts:
- moved R4 14.5 mm to (16.0, 33.5)
- moved R3 13.5 mm to (16.0, 31.0)
- moved U2 8.02 mm to (16.0, 27.5)
- moved A1 8.00 mm to (32.0, 30.1)
- moved A2 8.00 mm to (32.0, 30.1)
- moved A3 8.00 mm to (69.0, 30.1)
- moved C1 8.00 mm to (55.0, 40.0)
- moved R1 8.00 mm to (46.0, 22.0)
- moved R2 8.00 mm to (56.0, 22.0)
- moved U1 8.00 mm to (51.0, 26.0)
Routing:
- net GND1: track 316.5 -> 267.7 mm
- net VBUS1: track 127.5 -> 102.9 mm, vias 3 -> 1
- net USB_DM: track 74.4 -> 56.3 mm, vias 2 -> 1
- net USB_DP: track 70.7 -> 54.6 mm, vias 1 -> 3
- net CC1: track 14.6 -> 11.1 mm
- net CC2: track 15.1 -> 11.6 mm
- net SER_A2_B3: track 22.6 -> 20.4 mm
- net SER_A1_B0: track 20.5 -> 21.9 mm
Other:
- board size 88.8 x 58.9 mm -> 80.8 x 58.9 mm
